File: noritake_mn12864k_controller.kicad_pcb (KiCad board)
At the start: 4 copper layers, 99 x 46.5 mm, 187 parts, among them J1 Conn_01x11, J2 USB_C_Receptacle_USB2.0, J3 TagConnect_TC2030_SWD, J4 Conn_01x18, Q1 AO3400A, Q10 2N7002, Q11 LBSS84LT1G, Q12 2N7002, Q13 TO-252, Q14 CJT04N15, Q15 2N7002, Q16 LBSS84LT1G, Q17 2N7002, Q18 S9015, Q2 AO3400A, Q3 S9015, Q4 AO3401A, Q5 AO3401A, Q6 S9015, Q7 2N7002, Q8 LBSS84LT1G, Q9 2N7002, T1 Wuerth 760390013, T2 Wuerth 760390013, T3 Wuerth 760390013, T4 Wuerth 760390013, U1 SN74AVC8T245PW, U10 SRV05-4, U11 SRV05-4, U12 SRV05-4, U2 74HC14, U3 CD4051B, U4 MN12864K, U5 STM32F730R8T6, U6 NE555D, U7 74HC08, U8 SRV05-4, U9 XC6206PxxxMR

Commit message: Assign unique value to low voltage 0805 caps
Parts:
- C28, C29: value 10uF -> 10uF LV
Changed lines of the file:
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@@
       (drillshape 0)
       (scaleselection 1)
-      (outputdirectory "fab"))
+      (outputdirectory ""))
   )
   (net 0 "")
@@
       (effects (font (size 1 1) (thickness 0.15)))
     )
-    (fp_text value 10uF (at 0 1.68) (layer F.Fab)
+    (fp_text value "10uF LV" (at 0 1.68) (layer F.Fab)
       (effects (font (size 1 1) (thickness 0.15)))
     )
@@
       (effects (font (size 1 1) (thickness 0.15)))
     )
-    (fp_text value 10uF (at 0 1.68) (layer F.Fab)
+    (fp_text value "10uF LV" (at 0 1.68) (layer F.Fab)
       (effects (font (size 1 1) (thickness 0.15)))
     )
